File: PCB Designing/KiCAD/STM32F103Based/project1/project1.kicad_pcb (KiCad board)
At the start: 2 copper layers, 34.5 x 39.5 mm, 32 parts, among them J1 USB_B_Micro, J2 Conn_01x04_Pin, J3 Conn_01x04_Pin, J4 Conn_01x04_Pin, SW1 SW_SPDT, U1 STM32F103C8T6, U2 AMS1117-3.3, Y1 16MHz

Commit message: First PCB Complete
Parts:
- moved SW1 0.49 mm to (40.7, 38.0)
- moved J1 0.25 mm to (69.0, 45.6)
Routing:
- net +3.3V: track 10.8 -> 130.9 mm, vias 0 -> 6
- net GND: track 9.33 -> 35.4 mm, vias 0 -> 23
- net /NRST: track 0.00 -> 9.55 mm
- net /HSE_IN: track 3.92 -> 11.6 mm
- net +3.3VA: track 3.21 -> 6.39 mm
- net /PWR_LED_K: track 0.00 -> 2.74 mm
- net /HSE_OUT: track 3.89 -> 6.01 mm
- net /BOOT0: track 10.6 -> 11.9 mm
- added copper zone on F.Cu, net +3.3V
- added copper zone on F.Cu, net GND
- added copper zone on F.Cu, net VBUS
Other:
- board text added: "I2C2"
- board text added: "SWD"
- board text added: "USART1"
